Commit message: fix inertia-remove belt-set friction

File: urdf/base.xacro (robot description, xacro)
@@ -17,5 +17,5 @@
         </geometry>
       </collision>
-      <xacro:cylinder_inertial mass="0.005" radius="${radius}" length="0.01167"/>
+      <xacro:cylinder_inertial mass="1" radius="${radius}" length="0.01167"/>
     </link>
     <joint name="${link_name}_joint" type="continuous">
@@ -24,4 +24,5 @@
         <xacro:insert_block name="origin"/>
         <axis xyz="0 0 1"/>
+        <dynamics friction="1" damping="0"/>
     </joint>
     <transmission name="${link_name}_transmission">
@@ -35,25 +36,26 @@
         </actuator>
     </transmission>
-    <!-- <gazebo reference="${link_name}">
+    <gazebo reference="${link_name}">
       <selfCollide>true</selfCollide>
-      <mu1 value="200.0"/>
-      <mu2 value="100.0"/>
-      <kp value="10000000.0"/>
-      <kd value="1.0"/>
-    </gazebo> -->
+      <mu1 value="1"/>
+      <mu2 value="1"/>
+      <kp value="1000000.0"/>
+      <kd value="1"/>
+      <fdir1 value="0 0 1"/>
+    </gazebo>
   </xacro:macro>
 <xacro:wheel link_name="front_left_wheel" radius="0.01314">
-  <origin xyz="0.03 0.024 -0.012" rpy="${-pi/2} 0 0"/>
+  <origin xyz="0.03 0.024 -0.013" rpy="${-pi/2} 0 0"/>
 </xacro:wheel>
 <xacro:wheel link_name="front_right_wheel" radius="0.01314">
-  <origin xyz="0.03 -0.024 -0.012" rpy="${-pi/2} 0 0"/>
+  <origin xyz="0.03 -0.024 -0.013" rpy="${-pi/2} 0 0"/>
 </xacro:wheel>
-<xacro:wheel link_name="rear_left_wheel" radius="0.008995">
-  <origin xyz="-0.017 0.024 -0.0151707" rpy="${-pi/2} 0 0"/>
+<xacro:wheel link_name="rear_left_wheel" radius="0.01314">
+  <origin xyz="-0.017 0.024 -0.013" rpy="${-pi/2} 0 0"/>
 </xacro:wheel>
-<xacro:wheel link_name="rear_right_wheel" radius="0.008995">
-  <origin xyz="-0.017 -0.024 -0.0151707" rpy="${-pi/2} 0 0"/>
+<xacro:wheel link_name="rear_right_wheel" radius="0.01314">
+  <origin xyz="-0.017 -0.024 -0.013" rpy="${-pi/2} 0 0"/>
 </xacro:wheel>
-<link name="left_belt">
+<!-- <link name="left_belt">
   <visual>
     <geometry>
@@ -78,8 +80,8 @@
   <child link="right_belt"/>
   <origin xyz="0.00945088 -0.024 -0.0133211"/>
-</joint>
+</joint> -->
 <gazebo>
     <plugin name="skid_steer_drive_controller" filename="libgazebo_ros_skid_steer_drive.so">
-        <updateRate>25.0</updateRate>
+        <updateRate>100.0</updateRate>
         <robotNamespace>/</robotNamespace>
         <leftFrontJoint>front_left_wheel_joint</leftFrontJoint>
@@ -90,6 +92,6 @@
         <wheelDiameter>0.026281</wheelDiameter>
         <robotBaseFrame>base_footprint</robotBaseFrame>
-        <torque>0.1</torque>
-        <commandTopic>cmd_vel</commandTopic>
+        <torque>20</torque>
+        <commandTopic>vector/cmd_vel</commandTopic>
         <odometryTopic>odom</odometryTopic>
         <broadcastTF>true</broadcastTF>

File: urdf/inertia.xacro (robot description, xacro)
@@ -4,7 +4,7 @@
     <inertial>
       <mass value="${mass}" />
-      <inertia ixx="${0.0833333 * mass * (3 * radius * radius + length * length)}" ixy="0.0" ixz="0.0"
-        izz="${0.0833333 * mass * (3 * radius * radius + length * length)}" iyz="0.0"
-        iyy="${0.5 * mass * radius * radius}" />
+      <inertia ixx="${(1/4)*(mass)*(((1/3)*length*length)+(radius*radius))}" ixy="0.0" ixz="0.0"
+        iyy="${(1/4)*(mass)*(((1/3)*length*length)+(radius*radius))}" iyz="0.0"
+        izz="${0.5 * mass * radius * radius}" />
     </inertial>
   </xacro:macro>

File: urdf/vector.xacro (robot description, xacro)
@@ -11,5 +11,5 @@
   <!-- Body -->
   <link name="base_link">
-    <xacro:box_inertial mass="0.06" x="0.073" y="0.043" z="0.061" />
+    <xacro:box_inertial mass="0.05" x="0.073" y="0.043" z="0.061" />
     <visual>
       <geometry>
@@ -25,12 +25,12 @@
   <gazebo reference="base_link">
       <selfCollide>true</selfCollide>
-      <mu1 value="200.0"/>
-      <mu2 value="100.0"/>
-      <kp value="10000000.0"/>
+      <mu1 value="1"/>
+      <mu2 value="1"/>
+      <kp value="1000000.0"/>
       <kd value="1.0"/>
   </gazebo>
   <!-- Head -->
   <link name="head">
-    <xacro:box_inertial mass="0.01" x="0.036" y="0.038" z="0.041" />
+    <xacro:box_inertial mass="0.05" x="0.036" y="0.038" z="0.041" />
     <visual>
       <geometry>
@@ -45,13 +45,13 @@
   </link>
   <gazebo reference="head">
-      <kp>1000000000.0</kp>
-      <kd>1000000000.0</kd>
-      <mu1>10.0</mu1>
-      <mu2>10.0</mu2>
-      <self_collide>0</self_collide>
+      <kp>1000000.0</kp>
+      <kd>1.0</kd>
+      <mu1>1.0</mu1>
+      <mu2>1.0</mu2>
+      <self_collide>true</self_collide>
   </gazebo>
   <!-- lifter -->
   <link name="full_lift">
-    <xacro:box_inertial mass="0.01" x="0.081" y="0.058" z="0.050"/>
+    <xacro:box_inertial mass="0.05" x="0.081" y="0.058" z="0.050"/>
     <visual>
       <geometry>

Commit message: fix friction problem

File: urdf/base.xacro (robot description, xacro)
@@ -24,5 +24,4 @@
         <xacro:insert_block name="origin"/>
         <axis xyz="0 0 1"/>
-        <dynamics friction="1" damping="0"/>
     </joint>
     <transmission name="${link_name}_transmission">
@@ -42,5 +41,4 @@
       <kp value="1000000.0"/>
       <kd value="1"/>
-      <fdir1 value="0 0 1"/>
     </gazebo>
   </xacro:macro>
